Commit message: Push small changes from laptop

File: urdf/hand_ros.urdf (robot description, URDF)
Before this commit: robot visual, 16 links, 15 joints
Links:
- link base_link: geometry collision mesh filename=file:///home/patrick/contact/contact-sim/urdf/mesh/joint_0.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 scale=1 1 1; visual mesh filename=file:///home/patrick/contact/contact-sim/urdf/mesh/joint_0.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 scale=1 1 1
- link index_1: geometry collision mesh filename=file:///home/patrick/contact/contact-sim/urdf/mesh/joint_1.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 scale=1 1 1; visual mesh filename=file:///home/patrick/contact/contact-sim/urdf/mesh/joint_1.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 scale=1 1 1
- link index_2: geometry collision mesh filename=file:///home/patrick/contact/contact-sim/urdf/mesh/joint_2.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 scale=1 1 1; visual mesh filename=file:///home/patrick/contact/contact-sim/urdf/mesh/joint_2.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 scale=1 1 1
- link index_3: geometry collision mesh filename=file:///home/patrick/contact/contact-sim/urdf/mesh/joint_3.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 scale=1 1 1; visual mesh filename=file:///home/patrick/contact/contact-sim/urdf/mesh/joint_3.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 scale=1 1 1
- link middle_1: geometry collision mesh filename=file:///home/patrick/contact/contact-sim/urdf/mesh/joint_4.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 scale=1 1 1; visual mesh filename=file:///home/patrick/contact/contact-sim/urdf/mesh/joint_4.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 scale=1 1 1
- link middle_2: geometry collision mesh filename=file:///home/patrick/contact/contact-sim/urdf/mesh/joint_5.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 scale=1 1 1; visual mesh filename=file:///home/patrick/contact/contact-sim/urdf/mesh/joint_5.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 scale=1 1 1
- link middle_3: geometry collision mesh filename=file:///home/patrick/contact/contact-sim/urdf/mesh/joint_6.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 scale=1 1 1; visual mesh filename=file:///home/patrick/contact/contact-sim/urdf/mesh/joint_6.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 scale=1 1 1
- link pinky_1: geometry collision mesh filename=file:///home/patrick/contact/contact-sim/urdf/mesh/joint_7.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 scale=1 1 1; visual mesh filename=file:///home/patrick/contact/contact-sim/urdf/mesh/joint_7.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 scale=1 1 1
- link pinky_2: geometry collision mesh filename=file:///home/patrick/contact/contact-sim/urdf/mesh/joint_8.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 scale=1 1 1; visual mesh filename=file:///home/patrick/contact/contact-sim/urdf/mesh/joint_8.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 scale=1 1 1
- link pinky_3: geometry collision mesh filename=file:///home/patrick/contact/contact-sim/urdf/mesh/joint_9.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 scale=1 1 1; visual mesh filename=file:///home/patrick/contact/contact-sim/urdf/mesh/joint_9.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 scale=1 1 1
- link ring_1: geometry collision mesh filename=file:///home/patrick/contact/contact-sim/urdf/mesh/joint_10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 scale=1 1 1; visual mesh filename=file:///home/patrick/contact/contact-sim/urdf/mesh/joint_10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 scale=1 1 1
- link ring_2: geometry collision mesh filename=file:///home/patrick/contact/contact-sim/urdf/mesh/joint_11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 scale=1 1 1; visual mesh filename=file:///home/patrick/contact/contact-sim/urdf/mesh/joint_11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 scale=1 1 1
- link ring_3: geometry collision mesh filename=file:///home/patrick/contact/contact-sim/urdf/mesh/joint_12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 scale=1 1 1; visual mesh filename=file:///home/patrick/contact/contact-sim/urdf/mesh/joint_12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 scale=1 1 1
- link thumb_1: geometry collision mesh filename=file:///home/patrick/contact/contact-sim/urdf/mesh/joint_13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 scale=1 1 1; visual mesh filename=file:///home/patrick/contact/contact-sim/urdf/mesh/joint_13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 scale=1 1 1
- link thumb_2: geometry collision mesh filename=file:///home/patrick/contact/contact-sim/urdf/mesh/joint_14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 scale=1 1 1; visual mesh filename=file:///home/patrick/contact/contact-sim/urdf/mesh/joint_14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 scale=1 1 1
- link thumb_3: geometry collision mesh filename=file:///home/patrick/contact/contact-sim/urdf/mesh/joint_15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 scale=1 1 1; visual mesh filename=file:///home/patrick/contact/contact-sim/urdf/mesh/joint_15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 scale=1 1 1
