Commit message: Rudimentary human grasping working

File: urdf/hand.urdf (robot description, URDF)
Before this commit: robot visual, 4 links, 3 joints
Links:
- added link middle_1; collision mesh filename=/home/patrick/contact/contact-sim/mesh/joint_4.stl scale=1 1 1; visual mesh filename=/home/patrick/contact/contact-sim/mesh/joint_4.stl scale=1 1 1
- added link middle_2; collision mesh filename=/home/patrick/contact/contact-sim/mesh/joint_5.stl scale=1 1 1; visual mesh filename=/home/patrick/contact/contact-sim/mesh/joint_5.stl scale=1 1 1
- added link middle_3; collision mesh filename=/home/patrick/contact/contact-sim/mesh/joint_6.stl scale=1 1 1; visual mesh filename=/home/patrick/contact/contact-sim/mesh/joint_6.stl scale=1 1 1
- added link pinky_1; collision mesh filename=/home/patrick/contact/contact-sim/mesh/joint_7.stl scale=1 1 1; visual mesh filename=/home/patrick/contact/contact-sim/mesh/joint_7.stl scale=1 1 1
- added link pinky_2; collision mesh filename=/home/patrick/contact/contact-sim/mesh/joint_8.stl scale=1 1 1; visual mesh filename=/home/patrick/contact/contact-sim/mesh/joint_8.stl scale=1 1 1
- added link pinky_3; collision mesh filename=/home/patrick/contact/contact-sim/mesh/joint_9.stl scale=1 1 1; visual mesh filename=/home/patrick/contact/contact-sim/mesh/joint_9.stl scale=1 1 1
- added link ring_1; collision mesh filename=/home/patrick/contact/contact-sim/mesh/joint_10.stl scale=1 1 1; visual mesh filename=/home/patrick/contact/contact-sim/mesh/joint_10.stl scale=1 1 1
- added link ring_2; collision mesh filename=/home/patrick/contact/contact-sim/mesh/joint_11.stl scale=1 1 1; visual mesh filename=/home/patrick/contact/contact-sim/mesh/joint_11.stl scale=1 1 1
- added link ring_3; collision mesh filename=/home/patrick/contact/contact-sim/mesh/joint_12.stl scale=1 1 1; visual mesh filename=/home/patrick/contact/contact-sim/mesh/joint_12.stl scale=1 1 1
- added link thumb_1; collision mesh filename=/home/patrick/contact/contact-sim/mesh/joint_13.stl scale=1 1 1; visual mesh filename=/home/patrick/contact/contact-sim/mesh/joint_13.stl scale=1 1 1
- added link thumb_2; collision mesh filename=/home/patrick/contact/contact-sim/mesh/joint_14.stl scale=1 1 1; visual mesh filename=/home/patrick/contact/contact-sim/mesh/joint_14.stl scale=1 1 1
- added link thumb_3; collision mesh filename=/home/patrick/contact/contact-sim/mesh/joint_15.stl scale=1 1 1; visual mesh filename=/home/patrick/contact/contact-sim/mesh/joint_15.stl scale=1 1 1
- link base_link: geometry collision mesh filename=/home/patrick/contact/contact-sim/mesh/joint_0.stl scale=1 1 1; visual mesh filename=/home/patrick/contact/contact-sim/mesh/joint_0.stl scale=1 1 1
- link index_1: geometry collision mesh filename=/home/patrick/contact/contact-sim/mesh/joint_1.stl scale=1 1 1; visual mesh filename=/home/patrick/contact/contact-sim/mesh/joint_1.stl scale=1 1 1
- link index_2: geometry collision mesh filename=/home/patrick/contact/contact-sim/mesh/joint_2.stl scale=1 1 1; visual mesh filename=/home/patrick/contact/contact-sim/mesh/joint_2.stl scale=1 1 1
- link index_3: geometry collision mesh filename=/home/patrick/contact/contact-sim/mesh/joint_3.stl scale=1 1 1; visual mesh filename=/home/patrick/contact/contact-sim/mesh/joint_3.stl scale=1 1 1
Joints:
- added joint middle_1_to_middle_2: type revolute, parent middle_1, child middle_2, origin xyz=-0.0312 0.0019 -0.0056 rpy=-0.0773 -0.0436 0.2394, axis 0 0 1, limit lower=-1 upper=1 effort=1000.0 velocity=0.5
- added joint middle_2_to_middle_3: type revolute, parent middle_2, child middle_3, origin xyz=-0.0229 -0.0012 -0.0039 rpy=0.0009 0.0748 0.2820, axis 0 0 1, limit lower=-1 upper=1 effort=1000.0 velocity=0.5
- added joint palm_to_middle_1: type revolute, parent base_link, child middle_1, origin xyz=-0.0946 -0.0015 -0.0033 rpy=-0.0966 -0.1163 0.4734, axis 0 0 1, limit lower=-1 upper=1 effort=1000.0 velocity=0.5
- added joint palm_to_pinky_1: type revolute, parent base_link, child pinky_1, origin xyz=-0.0687 -0.0099 -0.0432 rpy=-0.9372 0.8386 1.3141, axis 0 0 1, limit lower=-1 upper=1 effort=1000.0 velocity=0.5
- added joint palm_to_ring_1: type revolute, parent base_link, child ring_1, origin xyz=-0.0817 -0.0040 -0.0267 rpy=-0.3148 0.1608 1.0260, axis 0 0 1, limit lower=-1 upper=1 effort=1000.0 velocity=0.5
- added joint palm_to_thumb_1: type revolute, parent base_link, child thumb_1, origin xyz=-0.0241 -0.0155 0.0258 rpy=0.7085 -0.0531 -0.1302, axis 0 0 1, limit lower=-1 upper=1 effort=1000.0 velocity=0.5
- added joint pinky_1_to_pinky_2: type revolute, parent pinky_1, child pinky_2, origin xyz=-0.0170 0.0001 -0.0125 rpy=0.4907 0.0007 0.4223, axis 0 0 1, limit lower=-1 upper=1 effort=1000.0 velocity=0.5
- added joint pinky_2_to_pinky_3: type revolute, parent pinky_2, child pinky_3, origin xyz=-0.0158 -0.0007 -0.0103 rpy=-0.6189 -0.1641 -0.2220, axis 0 0 1, limit lower=-1 upper=1 effort=1000.0 velocity=0.5
- added joint ring_1_to_ring_2: type revolute, parent ring_1, child ring_2, origin xyz=-0.0283 0.0021 -0.0051 rpy=-0.2046 0.0381 0.2742, axis 0 0 1, limit lower=-1 upper=1 effort=1000.0 velocity=0.5
- added joint ring_2_to_ring_3: type revolute, parent ring_2, child ring_3, origin xyz=-0.0235 -0.0017 -0.0076 rpy=-0.1173 0.1611 0.3245, axis 0 0 1, limit lower=-1 upper=1 effort=1000.0 velocity=0.5
- added joint thumb_1_to_thumb_2: type revolute, parent thumb_1, child thumb_2, origin xyz=-0.0196 0.0009 0.0237 rpy=-0.5732 0.1317 0.2807, axis 0 0 1, limit lower=-1 upper=1 effort=1000.0 velocity=0.5
- added joint thumb_2_to_thumb_3: type revolute, parent thumb_2, child thumb_3, origin xyz=-0.0222 -0.0054 0.0145 rpy=0.5888 -0.2052 -0.0819, axis 0 0 1, limit lower=-1 upper=1 effort=1000.0 velocity=0.5
- joint index_1_to_index_2: axis (none) -> 0 0 1; limit (none) -> lower=-1 upper=1 effort=1000.0 velocity=0.5; type continuous -> revolute
- joint index_2_to_index_3: axis (none) -> 0 0 1; limit (none) -> lower=-1 upper=1 effort=1000.0 velocity=0.5; type floating -> revolute
- joint palm_to_index_1: axis (none) -> 0 0 1; limit (none) -> lower=-1 upper=1 effort=1000.0 velocity=0.5; type continuous -> revolute

Commit message: Scripted hand generation, trying to get contact via deflection

File: urdf/hand.urdf (robot description, URDF)
Before this commit: robot visual, 16 links, 15 joints
Links:
- link base_link: geometry collision mesh filename=/home/patrick/contact/contact-sim/urdf/mesh/joint_0.stl scale=1 1 1; visual mesh filename=/home/patrick/contact/contact-sim/urdf/mesh/joint_0.stl scale=1 1 1
- link index_1: geometry collision mesh filename=/home/patrick/contact/contact-sim/urdf/mesh/joint_1.stl scale=1 1 1; visual mesh filename=/home/patrick/contact/contact-sim/urdf/mesh/joint_1.stl scale=1 1 1
- link index_2: geometry collision mesh filename=/home/patrick/contact/contact-sim/urdf/mesh/joint_2.stl scale=1 1 1; visual mesh filename=/home/patrick/contact/contact-sim/urdf/mesh/joint_2.stl scale=1 1 1
- link index_3: geometry collision mesh filename=/home/patrick/contact/contact-sim/urdf/mesh/joint_3.stl scale=1 1 1; visual mesh filename=/home/patrick/contact/contact-sim/urdf/mesh/joint_3.stl scale=1 1 1
- link middle_1: geometry collision mesh filename=/home/patrick/contact/contact-sim/urdf/mesh/joint_4.stl scale=1 1 1; visual mesh filename=/home/patrick/contact/contact-sim/urdf/mesh/joint_4.stl scale=1 1 1
- link middle_2: geometry collision mesh filename=/home/patrick/contact/contact-sim/urdf/mesh/joint_5.stl scale=1 1 1; visual mesh filename=/home/patrick/contact/contact-sim/urdf/mesh/joint_5.stl scale=1 1 1
- link middle_3: geometry collision mesh filename=/home/patrick/contact/contact-sim/urdf/mesh/joint_6.stl scale=1 1 1; visual mesh filename=/home/patrick/contact/contact-sim/urdf/mesh/joint_6.stl scale=1 1 1
- link pinky_1: geometry collision mesh filename=/home/patrick/contact/contact-sim/urdf/mesh/joint_7.stl scale=1 1 1; visual mesh filename=/home/patrick/contact/contact-sim/urdf/mesh/joint_7.stl scale=1 1 1
- link pinky_2: geometry collision mesh filename=/home/patrick/contact/contact-sim/urdf/mesh/joint_8.stl scale=1 1 1; visual mesh filename=/home/patrick/contact/contact-sim/urdf/mesh/joint_8.stl scale=1 1 1
- link pinky_3: geometry collision mesh filename=/home/patrick/contact/contact-sim/urdf/mesh/joint_9.stl scale=1 1 1; visual mesh filename=/home/patrick/contact/contact-sim/urdf/mesh/joint_9.stl scale=1 1 1
- link ring_1: geometry collision mesh filename=/home/patrick/contact/contact-sim/urdf/mesh/joint_10.stl scale=1 1 1; visual mesh filename=/home/patrick/contact/contact-sim/urdf/mesh/joint_10.stl scale=1 1 1
- link ring_2: geometry collision mesh filename=/home/patrick/contact/contact-sim/urdf/mesh/joint_11.stl scale=1 1 1; visual mesh filename=/home/patrick/contact/contact-sim/urdf/mesh/joint_11.stl scale=1 1 1
- link ring_3: geometry collision mesh filename=/home/patrick/contact/contact-sim/urdf/mesh/joint_12.stl scale=1 1 1; visual mesh filename=/home/patrick/contact/contact-sim/urdf/mesh/joint_12.stl scale=1 1 1
- link thumb_1: geometry collision mesh filename=/home/patrick/contact/contact-sim/urdf/mesh/joint_13.stl scale=1 1 1; visual mesh filename=/home/patrick/contact/contact-sim/urdf/mesh/joint_13.stl scale=1 1 1
- link thumb_2: geometry collision mesh filename=/home/patrick/contact/contact-sim/urdf/mesh/joint_14.stl scale=1 1 1; visual mesh filename=/home/patrick/contact/contact-sim/urdf/mesh/joint_14.stl scale=1 1 1
- link thumb_3: geometry collision mesh filename=/home/patrick/contact/contact-sim/urdf/mesh/joint_15.stl scale=1 1 1; visual mesh filename=/home/patrick/contact/contact-sim/urdf/mesh/joint_15.stl scale=1 1 1
Joints:
- joint index_1_to_index_2: origin xyz=-0.0327 0.0040 0.0022 rpy=-0.0144 -0.0299 0.1765 -> xyz=-0.0327 0.0040 0.0022 rpy=0.1225 0.0205 0.7585
- joint index_2_to_index_3: origin xyz=-0.0221 -0.0013 -0.0001 rpy=0.0407 0.0358 0.1450 -> xyz=-0.0221 -0.0013 -0.0001 rpy=-0.0876 0.0993 0.1844
- joint middle_1_to_middle_2: origin xyz=-0.0312 0.0019 -0.0056 rpy=-0.0773 -0.0436 0.2394 -> xyz=-0.0312 0.0019 -0.0056 rpy=-0.1508 -0.0021 0.7064
- joint middle_2_to_middle_3: origin xyz=-0.0229 -0.0012 -0.0039 rpy=0.0009 0.0748 0.2820 -> xyz=-0.0229 -0.0012 -0.0039 rpy=-0.0034 0.0938 0.3380
- joint palm_to_index_1: origin xyz=-0.0881 -0.0052 0.0207 rpy=0.1656 0.0305 0.1494 -> xyz=-0.0881 -0.0052 0.0207 rpy=0.0998 -0.0645 0.4137
- joint palm_to_middle_1: origin xyz=-0.0946 -0.0015 -0.0033 rpy=-0.0966 -0.1163 0.4734 -> xyz=-0.0946 -0.0015 -0.0033 rpy=-0.1258 -0.0180 0.5314
- joint palm_to_pinky_1: origin xyz=-0.0687 -0.0099 -0.0432 rpy=-0.9372 0.8386 1.3141 -> xyz=-0.0687 -0.0099 -0.0432 rpy=-0.3792 0.3168 0.5771
- joint palm_to_ring_1: origin xyz=-0.0817 -0.0040 -0.0267 rpy=-0.3148 0.1608 1.0260 -> xyz=-0.0817 -0.0040 -0.0267 rpy=-0.1066 0.1236 0.6304
- joint palm_to_thumb_1: origin xyz=-0.0241 -0.0155 0.0258 rpy=0.7085 -0.0531 -0.1302 -> xyz=-0.0241 -0.0155 0.0258 rpy=0.8613 -0.2811 -0.0316
- joint pinky_1_to_pinky_2: origin xyz=-0.0170 0.0001 -0.0125 rpy=0.4907 0.0007 0.4223 -> xyz=-0.0170 0.0001 -0.0125 rpy=-0.1899 0.1160 0.4980
- joint pinky_2_to_pinky_3: origin xyz=-0.0158 -0.0007 -0.0103 rpy=-0.6189 -0.1641 -0.2220 -> xyz=-0.0158 -0.0007 -0.0103 rpy=-0.3676 0.0735 0.0668
- joint ring_1_to_ring_2: origin xyz=-0.0283 0.0021 -0.0051 rpy=-0.2046 0.0381 0.2742 -> xyz=-0.0283 0.0021 -0.0051 rpy=-0.2674 0.1456 0.6167
- joint ring_2_to_ring_3: origin xyz=-0.0235 -0.0017 -0.0076 rpy=-0.1173 0.1611 0.3245 -> xyz=-0.0235 -0.0017 -0.0076 rpy=-0.1489 0.1611 0.3628
- joint thumb_1_to_thumb_2: origin xyz=-0.0196 0.0009 0.0237 rpy=-0.5732 0.1317 0.2807 -> xyz=-0.0196 0.0009 0.0237 rpy=-0.4991 -0.0384 -0.0442
- joint thumb_2_to_thumb_3: origin xyz=-0.0222 -0.0054 0.0145 rpy=0.5888 -0.2052 -0.0819 -> xyz=-0.0222 -0.0054 0.0145 rpy=0.5243 -0.1155 0.2532

Commit message: Updated many

File: urdf/hand.urdf (robot description, URDF)
Before this commit: robot visual, 16 links, 15 joints
Joints:
- joint index_1_to_index_2: axis 0 0 1 -> 0.1380 -0.0369 0.9897; origin xyz=-0.0327 0.0040 0.0022 rpy=0.1225 0.0205 0.7585 -> xyz=-0.0327 0.0040 0.0022 rpy=0.0000 0.0000 0.0000
- joint index_2_to_index_3: axis 0 0 1 -> -0.1161 0.4997 0.8584; origin xyz=-0.0221 -0.0013 -0.0001 rpy=-0.0876 0.0993 0.1844 -> xyz=-0.0222 -0.0013 -0.0001 rpy=0.0000 0.0000 0.0000
- joint middle_1_to_middle_2: axis 0 0 1 -> 0.0530 -0.0978 0.9938; origin xyz=-0.0312 0.0019 -0.0056 rpy=-0.1508 -0.0021 0.7064 -> xyz=-0.0312 0.0019 -0.0056 rpy=0.0000 0.0000 0.0000
- joint middle_2_to_middle_3: axis 0 0 1 -> 0.0621 0.1374 0.9886; origin xyz=-0.0229 -0.0012 -0.0039 rpy=-0.0034 0.0938 0.3380 -> xyz=-0.0229 -0.0013 -0.0039 rpy=0.0000 0.0000 0.0000
- joint palm_to_index_1: axis 0 0 1 -> 0.0573 -0.3832 0.9219; origin xyz=-0.0881 -0.0052 0.0207 rpy=0.0998 -0.0645 0.4137 -> xyz=-0.0881 -0.0052 0.0207 rpy=0.0000 0.0000 0.0000
- joint palm_to_middle_1: axis 0 0 1 -> -0.4354 -0.1759 0.8829; origin xyz=-0.0946 -0.0015 -0.0033 rpy=-0.1258 -0.0180 0.5314 -> xyz=-0.0947 -0.0015 -0.0034 rpy=0.0000 0.0000 0.0000
- joint palm_to_pinky_1: axis 0 0 1 -> -0.7138 0.1337 0.6875; origin xyz=-0.0687 -0.0099 -0.0432 rpy=-0.3792 0.3168 0.5771 -> xyz=-0.0688 -0.0099 -0.0432 rpy=0.0000 0.0000 0.0000
- joint palm_to_ring_1: axis 0 0 1 -> -0.3497 0.1281 0.9281; origin xyz=-0.0817 -0.0040 -0.0267 rpy=-0.1066 0.1236 0.6304 -> xyz=-0.0817 -0.0040 -0.0267 rpy=0.0000 0.0000 0.0000
- joint palm_to_thumb_1: axis 0 0 1 -> 0.7916 -0.5713 -0.2166; origin xyz=-0.0241 -0.0155 0.0258 rpy=0.8613 -0.2811 -0.0316 -> xyz=-0.0241 -0.0155 0.0258 rpy=0.0000 0.0000 0.0000
- joint pinky_1_to_pinky_2: axis 0 0 1 -> 0.2096 0.2490 0.9455; origin xyz=-0.0170 0.0001 -0.0125 rpy=-0.1899 0.1160 0.4980 -> xyz=-0.0170 0.0001 -0.0125 rpy=0.0000 0.0000 0.0000
- joint pinky_2_to_pinky_3: axis 0 0 1 -> -0.7858 -0.0810 0.6132; origin xyz=-0.0158 -0.0007 -0.0103 rpy=-0.3676 0.0735 0.0668 -> xyz=-0.0159 -0.0007 -0.0103 rpy=0.0000 0.0000 0.0000
- joint ring_1_to_ring_2: axis 0 0 1 -> -0.4653 0.2350 0.8534; origin xyz=-0.0283 0.0021 -0.0051 rpy=-0.2674 0.1456 0.6167 -> xyz=-0.0283 0.0021 -0.0051 rpy=0.0000 0.0000 0.0000
- joint ring_2_to_ring_3: axis 0 0 1 -> -0.2219 -0.0481 0.9739; origin xyz=-0.0235 -0.0017 -0.0076 rpy=-0.1489 0.1611 0.3628 -> xyz=-0.0235 -0.0017 -0.0076 rpy=0.0000 0.0000 0.0000
- joint thumb_1_to_thumb_2: axis 0 0 1 -> 0.7080 -0.7041 -0.0543; origin xyz=-0.0196 0.0009 0.0237 rpy=-0.4991 -0.0384 -0.0442 -> xyz=-0.0196 0.0009 0.0237 rpy=0.0000 0.0000 0.0000
- joint thumb_2_to_thumb_3: axis 0 0 1 -> 0.8481 -0.2952 -0.4399; origin xyz=-0.0222 -0.0054 0.0145 rpy=0.5243 -0.1155 0.2532 -> xyz=-0.0222 -0.0054 0.0145 rpy=0.0000 0.0000 0.0000

Commit message: Better batch processing

File: urdf/hand.urdf (robot description, URDF)
Before this commit: robot visual, 16 links, 15 joints
Joints:
- joint palm_to_thumb_1: limit lower=-1 upper=2 effort=1000.0 velocity=0.5 -> lower=-1 upper=1 effort=1000.0 velocity=0.5

Commit message: Changed URDF so STL origin is at the joint location

File: urdf/hand.urdf (robot description, URDF)
Before this commit: robot visual, 16 links, 15 joints
Joints:
- joint index_1_to_index_2: origin xyz=-0.0327 0.0040 0.0022 rpy=0.0000 0.0000 0.0000 -> xyz=-0.0327 0.0040 0.0022 rpy=0.1225 0.0205 0.7585
- joint index_2_to_index_3: origin xyz=-0.0222 -0.0013 -0.0001 rpy=0.0000 0.0000 0.0000 -> xyz=-0.0222 -0.0013 -0.0001 rpy=-0.0876 0.0993 0.1844
- joint middle_1_to_middle_2: origin xyz=-0.0312 0.0019 -0.0056 rpy=0.0000 0.0000 0.0000 -> xyz=-0.0312 0.0019 -0.0056 rpy=-0.1508 -0.0021 0.7064
- joint middle_2_to_middle_3: origin xyz=-0.0229 -0.0013 -0.0039 rpy=0.0000 0.0000 0.0000 -> xyz=-0.0229 -0.0013 -0.0039 rpy=-0.0034 0.0938 0.3380
- joint palm_to_index_1: origin xyz=-0.0881 -0.0052 0.0207 rpy=0.0000 0.0000 0.0000 -> xyz=-0.0881 -0.0052 0.0207 rpy=0.0998 -0.0645 0.4137
- joint palm_to_middle_1: origin xyz=-0.0947 -0.0015 -0.0034 rpy=0.0000 0.0000 0.0000 -> xyz=-0.0947 -0.0015 -0.0034 rpy=-0.1258 -0.0180 0.5314
- joint palm_to_pinky_1: origin xyz=-0.0688 -0.0099 -0.0432 rpy=0.0000 0.0000 0.0000 -> xyz=-0.0688 -0.0099 -0.0432 rpy=-0.3792 0.3168 0.5771
- joint palm_to_ring_1: origin xyz=-0.0817 -0.0040 -0.0267 rpy=0.0000 0.0000 0.0000 -> xyz=-0.0817 -0.0040 -0.0267 rpy=-0.1066 0.1236 0.6304
- joint palm_to_thumb_1: origin xyz=-0.0241 -0.0155 0.0258 rpy=0.0000 0.0000 0.0000 -> xyz=-0.0241 -0.0155 0.0258 rpy=0.8613 -0.2811 -0.0316
- joint pinky_1_to_pinky_2: origin xyz=-0.0170 0.0001 -0.0125 rpy=0.0000 0.0000 0.0000 -> xyz=-0.0170 0.0001 -0.0125 rpy=-0.1899 0.1160 0.4980
- joint pinky_2_to_pinky_3: origin xyz=-0.0159 -0.0007 -0.0103 rpy=0.0000 0.0000 0.0000 -> xyz=-0.0159 -0.0007 -0.0103 rpy=-0.3676 0.0735 0.0668
- joint ring_1_to_ring_2: origin xyz=-0.0283 0.0021 -0.0051 rpy=0.0000 0.0000 0.0000 -> xyz=-0.0283 0.0021 -0.0051 rpy=-0.2674 0.1456 0.6167
- joint ring_2_to_ring_3: origin xyz=-0.0235 -0.0017 -0.0076 rpy=0.0000 0.0000 0.0000 -> xyz=-0.0235 -0.0017 -0.0076 rpy=-0.1489 0.1611 0.3628
- joint thumb_1_to_thumb_2: origin xyz=-0.0196 0.0009 0.0237 rpy=0.0000 0.0000 0.0000 -> xyz=-0.0196 0.0009 0.0237 rpy=-0.4991 -0.0384 -0.0442
- joint thumb_2_to_thumb_3: origin xyz=-0.0222 -0.0054 0.0145 rpy=0.0000 0.0000 0.0000 -> xyz=-0.0222 -0.0054 0.0145 rpy=0.5243 -0.1155 0.2532

File: urdf/hand_ros.urdf (robot description, URDF)
Before this commit: robot visual, 16 links, 15 joints
Joints:
- joint index_1_to_index_2: origin xyz=-0.0327 0.0040 0.0022 rpy=0.0000 0.0000 0.0000 -> xyz=-0.0327 0.0040 0.0022 rpy=0.1225 0.0205 0.7585
- joint index_2_to_index_3: origin xyz=-0.0222 -0.0013 -0.0001 rpy=0.0000 0.0000 0.0000 -> xyz=-0.0222 -0.0013 -0.0001 rpy=-0.0876 0.0993 0.1844
- joint middle_1_to_middle_2: origin xyz=-0.0312 0.0019 -0.0056 rpy=0.0000 0.0000 0.0000 -> xyz=-0.0312 0.0019 -0.0056 rpy=-0.1508 -0.0021 0.7064
- joint middle_2_to_middle_3: origin xyz=-0.0229 -0.0013 -0.0039 rpy=0.0000 0.0000 0.0000 -> xyz=-0.0229 -0.0013 -0.0039 rpy=-0.0034 0.0938 0.3380
- joint palm_to_index_1: origin xyz=-0.0881 -0.0052 0.0207 rpy=0.0000 0.0000 0.0000 -> xyz=-0.0881 -0.0052 0.0207 rpy=0.0998 -0.0645 0.4137
- joint palm_to_middle_1: origin xyz=-0.0947 -0.0015 -0.0034 rpy=0.0000 0.0000 0.0000 -> xyz=-0.0947 -0.0015 -0.0034 rpy=-0.1258 -0.0180 0.5314
- joint palm_to_pinky_1: origin xyz=-0.0688 -0.0099 -0.0432 rpy=0.0000 0.0000 0.0000 -> xyz=-0.0688 -0.0099 -0.0432 rpy=-0.3792 0.3168 0.5771
- joint palm_to_ring_1: origin xyz=-0.0817 -0.0040 -0.0267 rpy=0.0000 0.0000 0.0000 -> xyz=-0.0817 -0.0040 -0.0267 rpy=-0.1066 0.1236 0.6304
- joint palm_to_thumb_1: limit lower=-1 upper=2 effort=1000.0 velocity=0.5 -> lower=-1 upper=1 effort=1000.0 velocity=0.5; origin xyz=-0.0241 -0.0155 0.0258 rpy=0.0000 0.0000 0.0000 -> xyz=-0.0241 -0.0155 0.0258 rpy=0.8613 -0.2811 -0.0316
- joint pinky_1_to_pinky_2: origin xyz=-0.0170 0.0001 -0.0125 rpy=0.0000 0.0000 0.0000 -> xyz=-0.0170 0.0001 -0.0125 rpy=-0.1899 0.1160 0.4980
- joint pinky_2_to_pinky_3: origin xyz=-0.0159 -0.0007 -0.0103 rpy=0.0000 0.0000 0.0000 -> xyz=-0.0159 -0.0007 -0.0103 rpy=-0.3676 0.0735 0.0668
- joint ring_1_to_ring_2: origin xyz=-0.0283 0.0021 -0.0051 rpy=0.0000 0.0000 0.0000 -> xyz=-0.0283 0.0021 -0.0051 rpy=-0.2674 0.1456 0.6167
- joint ring_2_to_ring_3: origin xyz=-0.0235 -0.0017 -0.0076 rpy=0.0000 0.0000 0.0000 -> xyz=-0.0235 -0.0017 -0.0076 rpy=-0.1489 0.1611 0.3628
- joint thumb_1_to_thumb_2: origin xyz=-0.0196 0.0009 0.0237 rpy=0.0000 0.0000 0.0000 -> xyz=-0.0196 0.0009 0.0237 rpy=-0.4991 -0.0384 -0.0442
- joint thumb_2_to_thumb_3: origin xyz=-0.0222 -0.0054 0.0145 rpy=0.0000 0.0000 0.0000 -> xyz=-0.0222 -0.0054 0.0145 rpy=0.5243 -0.1155 0.2532
