Commit message: Back to flat hand mean

File: urdf/hand.urdf (robot description, URDF)
Before this commit: robot visual, 16 links, 15 joints
Joints:
- joint index_1_to_index_2: origin xyz=-0.0327 0.0040 0.0022 rpy=0.1225 0.0205 0.7585 -> xyz=-0.0327 0.0040 0.0022 rpy=0.0000 0.0000 0.0000
- joint index_2_to_index_3: origin xyz=-0.0222 -0.0013 -0.0001 rpy=-0.0876 0.0993 0.1844 -> xyz=-0.0222 -0.0013 -0.0001 rpy=0.0000 0.0000 0.0000
- joint middle_1_to_middle_2: origin xyz=-0.0312 0.0019 -0.0056 rpy=-0.1508 -0.0021 0.7064 -> xyz=-0.0312 0.0019 -0.0056 rpy=0.0000 0.0000 0.0000
- joint middle_2_to_middle_3: origin xyz=-0.0229 -0.0013 -0.0039 rpy=-0.0034 0.0938 0.3380 -> xyz=-0.0229 -0.0013 -0.0039 rpy=0.0000 0.0000 0.0000
- joint palm_to_index_1: origin xyz=-0.0881 -0.0052 0.0207 rpy=0.0998 -0.0645 0.4137 -> xyz=-0.0881 -0.0052 0.0207 rpy=0.0000 0.0000 0.0000
- joint palm_to_middle_1: origin xyz=-0.0947 -0.0015 -0.0034 rpy=-0.1258 -0.0180 0.5314 -> xyz=-0.0947 -0.0015 -0.0034 rpy=0.0000 0.0000 0.0000
- joint palm_to_pinky_1: origin xyz=-0.0688 -0.0099 -0.0432 rpy=-0.3792 0.3168 0.5771 -> xyz=-0.0688 -0.0099 -0.0432 rpy=0.0000 0.0000 0.0000
- joint palm_to_ring_1: origin xyz=-0.0817 -0.0040 -0.0267 rpy=-0.1066 0.1236 0.6304 -> xyz=-0.0817 -0.0040 -0.0267 rpy=0.0000 0.0000 0.0000
- joint palm_to_thumb_1: origin xyz=-0.0241 -0.0155 0.0258 rpy=0.8613 -0.2811 -0.0316 -> xyz=-0.0241 -0.0155 0.0258 rpy=0.0000 0.0000 0.0000
- joint pinky_1_to_pinky_2: origin xyz=-0.0170 0.0001 -0.0125 rpy=-0.1899 0.1160 0.4980 -> xyz=-0.0170 0.0001 -0.0125 rpy=0.0000 0.0000 0.0000
- joint pinky_2_to_pinky_3: origin xyz=-0.0159 -0.0007 -0.0103 rpy=-0.3676 0.0735 0.0668 -> xyz=-0.0159 -0.0007 -0.0103 rpy=0.0000 0.0000 0.0000
- joint ring_1_to_ring_2: origin xyz=-0.0283 0.0021 -0.0051 rpy=-0.2674 0.1456 0.6167 -> xyz=-0.0283 0.0021 -0.0051 rpy=0.0000 0.0000 0.0000
- joint ring_2_to_ring_3: origin xyz=-0.0235 -0.0017 -0.0076 rpy=-0.1489 0.1611 0.3628 -> xyz=-0.0235 -0.0017 -0.0076 rpy=0.0000 0.0000 0.0000
- joint thumb_1_to_thumb_2: origin xyz=-0.0196 0.0009 0.0237 rpy=-0.4991 -0.0384 -0.0442 -> xyz=-0.0196 0.0009 0.0237 rpy=0.0000 0.0000 0.0000
- joint thumb_2_to_thumb_3: origin xyz=-0.0222 -0.0054 0.0145 rpy=0.5243 -0.1155 0.2532 -> xyz=-0.0222 -0.0054 0.0145 rpy=0.0000 0.0000 0.0000

File: urdf/hand_ros.urdf (robot description, URDF)
Before this commit: robot visual, 16 links, 15 joints
Joints:
- joint index_1_to_index_2: origin xyz=-0.0327 0.0040 0.0022 rpy=0.1225 0.0205 0.7585 -> xyz=-0.0327 0.0040 0.0022 rpy=0.0000 0.0000 0.0000
- joint index_2_to_index_3: origin xyz=-0.0222 -0.0013 -0.0001 rpy=-0.0876 0.0993 0.1844 -> xyz=-0.0222 -0.0013 -0.0001 rpy=0.0000 0.0000 0.0000
- joint middle_1_to_middle_2: origin xyz=-0.0312 0.0019 -0.0056 rpy=-0.1508 -0.0021 0.7064 -> xyz=-0.0312 0.0019 -0.0056 rpy=0.0000 0.0000 0.0000
- joint middle_2_to_middle_3: origin xyz=-0.0229 -0.0013 -0.0039 rpy=-0.0034 0.0938 0.3380 -> xyz=-0.0229 -0.0013 -0.0039 rpy=0.0000 0.0000 0.0000
- joint palm_to_index_1: origin xyz=-0.0881 -0.0052 0.0207 rpy=0.0998 -0.0645 0.4137 -> xyz=-0.0881 -0.0052 0.0207 rpy=0.0000 0.0000 0.0000
- joint palm_to_middle_1: origin xyz=-0.0947 -0.0015 -0.0034 rpy=-0.1258 -0.0180 0.5314 -> xyz=-0.0947 -0.0015 -0.0034 rpy=0.0000 0.0000 0.0000
- joint palm_to_pinky_1: origin xyz=-0.0688 -0.0099 -0.0432 rpy=-0.3792 0.3168 0.5771 -> xyz=-0.0688 -0.0099 -0.0432 rpy=0.0000 0.0000 0.0000
- joint palm_to_ring_1: origin xyz=-0.0817 -0.0040 -0.0267 rpy=-0.1066 0.1236 0.6304 -> xyz=-0.0817 -0.0040 -0.0267 rpy=0.0000 0.0000 0.0000
- joint palm_to_thumb_1: origin xyz=-0.0241 -0.0155 0.0258 rpy=0.8613 -0.2811 -0.0316 -> xyz=-0.0241 -0.0155 0.0258 rpy=0.0000 0.0000 0.0000
- joint pinky_1_to_pinky_2: origin xyz=-0.0170 0.0001 -0.0125 rpy=-0.1899 0.1160 0.4980 -> xyz=-0.0170 0.0001 -0.0125 rpy=0.0000 0.0000 0.0000
- joint pinky_2_to_pinky_3: origin xyz=-0.0159 -0.0007 -0.0103 rpy=-0.3676 0.0735 0.0668 -> xyz=-0.0159 -0.0007 -0.0103 rpy=0.0000 0.0000 0.0000
- joint ring_1_to_ring_2: origin xyz=-0.0283 0.0021 -0.0051 rpy=-0.2674 0.1456 0.6167 -> xyz=-0.0283 0.0021 -0.0051 rpy=0.0000 0.0000 0.0000
- joint ring_2_to_ring_3: origin xyz=-0.0235 -0.0017 -0.0076 rpy=-0.1489 0.1611 0.3628 -> xyz=-0.0235 -0.0017 -0.0076 rpy=0.0000 0.0000 0.0000
- joint thumb_1_to_thumb_2: origin xyz=-0.0196 0.0009 0.0237 rpy=-0.4991 -0.0384 -0.0442 -> xyz=-0.0196 0.0009 0.0237 rpy=0.0000 0.0000 0.0000
- joint thumb_2_to_thumb_3: origin xyz=-0.0222 -0.0054 0.0145 rpy=0.5243 -0.1155 0.2532 -> xyz=-0.0222 -0.0054 0.0145 rpy=0.0000 0.0000 0.0000

Commit message: Manual tweak to hand joint axes to make fingers overlap less

File: urdf/hand.urdf (robot description, URDF)
Before this commit: robot visual, 16 links, 15 joints
Joints:
- joint palm_to_index_1: axis 0.0573 -0.3832 0.9219 -> 0.0573 -0.1832 0.9219
- joint palm_to_ring_1: axis -0.3497 0.1281 0.9281 -> -0.2497 0.1081 0.9281
